Commit message: fix urdf include path

File: turtlebot2_description/robots/kobuki_hexagons_hokuyo.urdf.xacro (robot description, xacro)
@@ -1,9 +1,9 @@
 <?xml version="1.0"?>
 <robot name="turtlebot" xmlns:xacro="http://ros.org/wiki/xacro">
-  <xacro:include filename="$(find turtlebot_description)/urdf/turtlebot_common_library.urdf.xacro" />
+  <xacro:include filename="$(find turtlebot2_description)/urdf/turtlebot_common_library.urdf.xacro" />
   <xacro:include filename="$(find kobuki_description)/urdf/kobuki.urdf.xacro" />
-  <xacro:include filename="$(find turtlebot_description)/urdf/stacks/hexagons.urdf.xacro" />
+  <xacro:include filename="$(find turtlebot2_description)/urdf/stacks/hexagons.urdf.xacro" />
   <!-- <xacro:include filename="$(find turtlebot_description)/urdf/sensors/kinect.urdf.xacro"/> -->
-  <xacro:include filename="$(find turtlebot_description)/urdf/sensors/hokuyo.urdf.xacro" />
+  <xacro:include filename="$(find turtlebot2_description)/urdf/sensors/hokuyo.urdf.xacro" />
   <xacro:kobuki />
   <xacro:stack_hexagons parent="base_link" />

File: turtlebot2_description/urdf/sensors/hokuyo.urdf.xacro (robot description, xacro)
@@ -1,6 +1,6 @@
 <?xml version="1.0"?>
 <robot name="sensor_hokuyo" xmlns:xacro="http://ros.org/wiki/xacro">
-    <xacro:include filename="$(find turtlebot_description)/urdf/turtlebot_gazebo.urdf.xacro" />
-    <xacro:include filename="$(find turtlebot_description)/urdf/turtlebot_properties.urdf.xacro" />
+    <xacro:include filename="$(find turtlebot2_description)/urdf/turtlebot_gazebo.urdf.xacro" />
+    <xacro:include filename="$(find turtlebot2_description)/urdf/turtlebot_properties.urdf.xacro" />
     <xacro:property name="laser_px" value="0.1" />
     <xacro:property name="laser_py" value="0" />

File: turtlebot2_description/urdf/stacks/hexagons.urdf.xacro (robot description, xacro)
@@ -4,5 +4,5 @@
  -->
 <robot name="stack_hexagons" xmlns:xacro="http://ros.org/wiki/xacro">
-  <xacro:include filename="$(find turtlebot_description)/urdf/common_properties.urdf.xacro"/>
+  <xacro:include filename="$(find turtlebot2_description)/urdf/common_properties.urdf.xacro"/>
   <!-- Xacro properties -->
   <xacro:property name="M_SCALE" value="0.001"/>
@@ -19,5 +19,5 @@
         <origin xyz="0 0 0" rpy="0 0 0"/>
         <geometry>
-          <mesh filename="package://turtlebot_description/meshes/stacks/hexagons/pole_bottom.dae"/>
+          <mesh filename="package://turtlebot2_description/meshes/stacks/hexagons/pole_bottom.dae"/>
         </geometry>
       </visual>
@@ -47,5 +47,5 @@
         <origin xyz="0 0 0" rpy="0 ${M_PI} 0"/>
         <geometry>
-          <mesh filename="package://turtlebot_description/meshes/stacks/hexagons/pole_middle.dae"/>
+          <mesh filename="package://turtlebot2_description/meshes/stacks/hexagons/pole_middle.dae"/>
         </geometry>
       </visual>
@@ -75,5 +75,5 @@
         <origin xyz=" 0 0 0" rpy="0 0 0"/>
         <geometry>
-          <mesh filename="package://turtlebot_description/meshes/stacks/hexagons/pole_top.dae"/>
+          <mesh filename="package://turtlebot2_description/meshes/stacks/hexagons/pole_top.dae"/>
         </geometry>
       </visual>
@@ -103,5 +103,5 @@
         <origin xyz="0 0 0" rpy="0 0 0"/>
         <geometry>
-          <mesh filename="package://turtlebot_description/meshes/stacks/hexagons/pole_kinect.dae" />
+          <mesh filename="package://turtlebot2_description/meshes/stacks/hexagons/pole_kinect.dae" />
         </geometry>
       </visual>
@@ -142,5 +142,5 @@
         <origin xyz="0 0 0" rpy="0 0 0"/>
         <geometry>
-          <mesh filename="package://turtlebot_description/meshes/stacks/hexagons/plate_bottom.dae"/>
+          <mesh filename="package://turtlebot2_description/meshes/stacks/hexagons/plate_bottom.dae"/>
         </geometry>
       </visual>
@@ -172,5 +172,5 @@
         <origin xyz="0 0 0" rpy="0 0 0"/>
         <geometry>
-          <mesh filename="package://turtlebot_description/meshes/stacks/hexagons/plate_middle.dae"/>
+          <mesh filename="package://turtlebot2_description/meshes/stacks/hexagons/plate_middle.dae"/>
         </geometry>
       </visual>
@@ -178,5 +178,5 @@
         <origin xyz="0.01364 0.0 0.0" rpy="0 0 0"/>
         <geometry>
-          <mesh filename="package://turtlebot_description/meshes/stacks/hexagons/plate_simple-binary.stl"
+          <mesh filename="package://turtlebot2_description/meshes/stacks/hexagons/plate_simple-binary.stl"
                 scale="${M_SCALE} ${M_SCALE} ${M_SCALE}"/>
         </geometry>
@@ -205,5 +205,5 @@
         <origin xyz="0 0 0" rpy="0 0 0"/>
         <geometry>
-          <mesh filename="package://turtlebot_description/meshes/stacks/hexagons/plate_top.dae"/>
+          <mesh filename="package://turtlebot2_description/meshes/stacks/hexagons/plate_top.dae"/>
         </geometry>
       </visual>
@@ -211,5 +211,5 @@
         <origin xyz="0.01364 0 0" rpy="0 0 0"/>
         <geometry>
-          <mesh filename="package://turtlebot_description/meshes/stacks/hexagons/plate_simple-binary.stl"
+          <mesh filename="package://turtlebot2_description/meshes/stacks/hexagons/plate_simple-binary.stl"
                 scale="${M_SCALE} ${M_SCALE} ${M_SCALE}"/>
         </geometry>

File: turtlebot2_description/urdf/turtlebot_common_library.urdf.xacro (robot description, xacro)
@@ -5,5 +5,5 @@
 <robot xmlns:xacro="http://ros.org/wiki/xacro">
   <!-- General -->
-  <xacro:include filename="$(find turtlebot_description)/urdf/common_properties.urdf.xacro"/>
-  <xacro:include filename="$(find turtlebot_description)/urdf/turtlebot_properties.urdf.xacro"/>
+  <xacro:include filename="$(find turtlebot2_description)/urdf/common_properties.urdf.xacro"/>
+  <xacro:include filename="$(find turtlebot2_description)/urdf/turtlebot_properties.urdf.xacro"/>
 </robot>
