Commit message: first slam configuration

File: turtlebot2_description/robots/tmp.urdf (robot description, URDF)
Before this commit: robot turtlebot, 30 links, 29 joints
Links:
- link laser: geometry collision box size=0.05 0.05 0.05; visual box size=0.05 0.05 0.05
Joints:
- joint laser_joint: origin xyz=0.1 0 0.24 rpy=0 0 0 -> xyz=0.1 0 0.21 rpy=0 0 0

File: turtlebot2_description/urdf/sensors/hokuyo.urdf.xacro (robot description, xacro)
@@ -5,5 +5,5 @@
     <xacro:property name="laser_px" value="0.1" />
     <xacro:property name="laser_py" value="0" />
-    <xacro:property name="laser_pz" value="0.24" />
+    <xacro:property name="laser_pz" value="0.21" />
     <xacro:macro name="box_inertia" params="x y z mass">
         <inertia ixx="${0.0833333 * mass * (y*y + z*z)}" ixy="0.0" ixz="0.0" iyy="${0.0833333 * mass * (x*x + z*z)}" iyz="0.0" izz="${0.0833333 * mass * (x*x + y*y)}" />
@@ -22,10 +22,10 @@
                 <origin xyz="0 0 0" rpy="0 0 0" />
                 <mass value="0.2" />
-                <xacro:box_inertia x="0.05" y="0.05" z="0.08" mass="0.2" />
+                <xacro:box_inertia x="0.05" y="0.05" z="0.05" mass="0.2" />
             </inertial>
             <visual>
                 <origin xyz="0 0 0" rpy="0 0 0" />
                 <geometry>
-                    <box size="0.05 0.05 0.08" />
+                    <box size="0.05 0.05 0.05" />
                 </geometry>
                 <material name="orange" />
@@ -35,8 +35,45 @@
                 <geometry>
                     <!-- <cylinder radius="0.1" length="0.2" /> -->
-                    <box size="0.05 0.05 0.08" />
+                    <box size="0.05 0.05 0.05" />
                 </geometry>
             </collision>
         </link>
+        <gazebo reference="laser">
+            <sensor type="ray" name="head_hokuyo_sensor">
+                <pose>0 0 0 0 0 0</pose>
+                <visualize>true</visualize>
+                <update_rate>20</update_rate>
+                <ray>
+                    <scan>
+                        <horizontal>
+                            <samples>720</samples>
+                            <resolution>1</resolution>
+                            <min_angle>-2.355</min_angle>
+                            <max_angle>2.355</max_angle>
+                        </horizontal>
+                    </scan>
+                    <range>
+                        <min>0.10</min>
+                        <max>5.0</max>
+                        <resolution>0.01</resolution>
+                    </range>
+                    <noise>
+                        <type>gaussian</type>
+                        <mean>0.0</mean>
+                        <stddev>0.01</stddev>
+                    </noise>
+                </ray>
+                <plugin name="turtlebot2_laserscan" filename="libgazebo_ros_ray_sensor.so">
+                    <ros>
+                      <remapping>~/out:=scan</remapping>
+                    </ros>
+                    <output_type>sensor_msgs/LaserScan</output_type>
+                    <frame_name>laser</frame_name>
+                  </plugin>
+            </sensor>
+        </gazebo>
+        <gazebo reference="laser">
+            <material>Gazebo/Orange</material>
+        </gazebo>
     </xacro:macro>
 </robot>
