Commit message: small refactor

File: turtlebot2_description/urdf/sensors/hokuyo.urdf.xacro (robot description, xacro)
@@ -6,4 +6,5 @@
     <xacro:property name="laser_py" value="0" />
     <xacro:property name="laser_pz" value="0.21" />
+    <xacro:property name="robot_namespace" value="/tb2_5"/>
     <xacro:macro name="box_inertia" params="x y z mass">
         <inertia ixx="${0.0833333 * mass * (y*y + z*z)}" ixy="0.0" ixz="0.0" iyy="${0.0833333 * mass * (x*x + z*z)}" iyz="0.0" izz="${0.0833333 * mass * (x*x + y*y)}" />
@@ -34,5 +35,4 @@
                 <origin xyz="0 0 0" rpy="0 0 0" />
                 <geometry>
-                    <!-- <cylinder radius="0.1" length="0.2" /> -->
                     <box size="0.05 0.05 0.05" />
                 </geometry>
@@ -69,6 +69,5 @@
                     <ros>
                       <remapping>~/out:=scan</remapping>
-                      <!-- TODO! AUTOMATIC NAMESPACE -->
-		              <namespace>/tb2</namespace>
+		              <namespace>${robot_namespace}</namespace>
                     </ros>
                     <output_type>sensor_msgs/LaserScan</output_type>

Commit message: Add Gazebo TB2 simulation

File: turtlebot2_description/urdf/sensors/hokuyo.urdf.xacro (robot description, xacro)
@@ -5,5 +5,6 @@
     <xacro:property name="laser_px" value="0.1" />
     <xacro:property name="laser_py" value="0" />
-    <xacro:property name="laser_pz" value="0.24" />
+    <xacro:property name="laser_pz" value="0.21" />
+    <xacro:property name="robot_namespace" value="/tb2_5"/>
     <xacro:macro name="box_inertia" params="x y z mass">
         <inertia ixx="${0.0833333 * mass * (y*y + z*z)}" ixy="0.0" ixz="0.0" iyy="${0.0833333 * mass * (x*x + z*z)}" iyz="0.0" izz="${0.0833333 * mass * (x*x + y*y)}" />
@@ -22,10 +23,10 @@
                 <origin xyz="0 0 0" rpy="0 0 0" />
                 <mass value="0.2" />
-                <xacro:box_inertia x="0.05" y="0.05" z="0.08" mass="0.2" />
+                <xacro:box_inertia x="0.05" y="0.05" z="0.05" mass="0.2" />
             </inertial>
             <visual>
                 <origin xyz="0 0 0" rpy="0 0 0" />
                 <geometry>
-                    <box size="0.05 0.05 0.08" />
+                    <box size="0.05 0.05 0.05" />
                 </geometry>
                 <material name="orange" />
@@ -34,9 +35,48 @@
                 <origin xyz="0 0 0" rpy="0 0 0" />
                 <geometry>
-                    <!-- <cylinder radius="0.1" length="0.2" /> -->
-                    <box size="0.05 0.05 0.08" />
+                    <box size="0.05 0.05 0.05" />
                 </geometry>
             </collision>
         </link>
+        <gazebo reference="laser">
+            <sensor type="ray" name="head_hokuyo_sensor">
+                <pose>0 0 0 0 0 0</pose>
+                <visualize>true</visualize>
+                <update_rate>20</update_rate>
+                <ray>
+                    <scan>
+                        <horizontal>
+                            <samples>720</samples>
+                            <resolution>1</resolution>
+                            <!-- <min_angle>-2.355</min_angle>
+                            <max_angle>2.355</max_angle> -->
+                            <min_angle>-1.56</min_angle>
+                            <max_angle>1.56</max_angle>
+                        </horizontal>
+                    </scan>
+                    <range>
+                        <min>0.10</min>
+                        <max>10.0</max>
+                        <resolution>0.01</resolution>
+                    </range>
+                    <noise>
+                        <type>gaussian</type>
+                        <mean>0.0</mean>
+                        <stddev>0.01</stddev>
+                    </noise>
+                </ray>
+                <plugin name="turtlebot2_laserscan" filename="libgazebo_ros_ray_sensor.so">
+                    <ros>
+                      <remapping>~/out:=scan</remapping>
+		              <namespace>${robot_namespace}</namespace>
+                    </ros>
+                    <output_type>sensor_msgs/LaserScan</output_type>
+                    <frame_name>laser</frame_name>
+                  </plugin>
+            </sensor>
+        </gazebo>
+        <gazebo reference="laser">
+            <material>Gazebo/Orange</material>
+        </gazebo>
     </xacro:macro>
 </robot>

Commit message: add automatic namespace in yaml and rviz and xacro

File: turtlebot2_description/urdf/sensors/hokuyo.urdf.xacro (robot description, xacro)
@@ -6,5 +6,6 @@
     <xacro:property name="laser_py" value="0" />
     <xacro:property name="laser_pz" value="0.21" />
-    <xacro:property name="robot_namespace" value="/tb2_5"/>
+    <xacro:arg name="namespace" default=""/>
+    <xacro:property name="robot_namespace" value="/$(arg namespace)"/>
     <xacro:macro name="box_inertia" params="x y z mass">
         <inertia ixx="${0.0833333 * mass * (y*y + z*z)}" ixy="0.0" ixz="0.0" iyy="${0.0833333 * mass * (x*x + z*z)}" iyz="0.0" izz="${0.0833333 * mass * (x*x + y*y)}" />
